File: lsw.kicad_sch (KiCad schematic)
At the start: 12 parts, among them Q2 FDN 306P, Q3 NMOS, U3 TPS2553DBVT-1

Commit message: Almost ready for production
Parts:
- C26: LCSC (none) -> C48579599
- D5, D6: LCSC (none) -> C5144142
- D7: LCSC (none) -> C84260
- Q2: LCSC (none) -> C154510
- Q3: footprint Package_TO_SOT_SMD:SOT-23-3 -> Package_TO_SOT_SMD:SOT-23; LCSC (none) -> C145103
- R5, R7: LCSC (none) -> C3009137
- R6: LCSC (none) -> C95781
- R8: LCSC (none) -> C17455
- R9: LCSC (none) -> C114523
- U3: LCSC (none) -> C2680358
