File: radio_mcu.kicad_sch (KiCad schematic)
At the start: 30 parts, among them J3 Conn_01x03_Pin, Q1 ???, Q4 Q_NPN, U1 STM32WL55CCU7, X1 32MHz

Commit message: Finalize design
Parts:
- removed D8: Green, LED_SMD:LED_0805_2012Metric, symbol Device:LED
- removed Q1: ???, Package_TO_SOT_SMD:SOT-23, symbol Transistor_FET:NDT3055L
- removed R13: 470, Resistor_SMD:R_0805_2012Metric, symbol Device:R
- added D5, D6: Green, LED_SMD:LED_0805_2012Metric, symbol Device:LED
- added Q2: DMN1019USN-7, Package_TO_SOT_SMD:SOT-23, symbol Transistor_FET:DMN10H220L
- added R5, R6: 470, Resistor_SMD:R_0805_2012Metric, symbol Device:R
Connections:
- net GND: now also Q2.2 (S), R5.2, R6.2
- net RF out/RX_EN: now also D5.2 (A)
- net RF out/TX_EN: now also D6.2 (A)
- net UART: now also Q2.3 (D)
- net UART2_TX: now also Q2.1 (G)
- net VBAT: now also R11.2; no longer Q4.3 (C)
- net at R10.1, U1.1 (PB3): now also Q4.2 (E); no longer R11.1
- new net: D6.1 (K), R6.1
- new net: D5.1 (K), R5.1
- new net: Q4.3 (C), R11.1
Other:
- removed sheet LSW
- moved on the sheet: R11

Commit message: Altered LCSC part numbers according to current stock
Parts:
- C1, C9: footprint Capacitor_SMD:C_0603_1608Metric -> Capacitor_SMD:C_0805_2012Metric; LCSC C49326648 -> C13967
- C2: value 1n -> 12p; LCSC C49326696 -> C1792
- C7, C8: LCSC C48579643 -> C13967
- U1: LCSC C3606913 -> C5270474
- X1: LCSC C2650719 -> C9009
Changed lines of the file:
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@@
 			)
 		)
-		(property "LCSC" "C3606913"
+		(property "LCSC" "C5270474"
 			(at 127 82.55 0)
 			(effects
@@
 			)
 		)
-		(property "Value" "1n"
+		(property "Value" "12p"
 			(at 55.88 62.2299 0)
 			(effects
@@
 			)
 		)
-		(property "LCSC" "C49326696"
+		(property "LCSC" "C1792"
 			(at 52.07 60.96 0)
 			(effects
@@
 			)
 		)
-		(property "Footprint" "Capacitor_SMD:C_0603_1608Metric"
+		(property "Footprint" "Capacitor_SMD:C_0805_2012Metric"
 			(at 46.6852 161.29 0)
 			(effects
@@
 			)
 		)
-		(property "LCSC" "C49326648"
+		(property "LCSC" "C13967"
 			(at 45.72 157.48 0)
 			(effects
@@
 			)
 		)
-		(property "Footprint" "Capacitor_SMD:C_0603_1608Metric"
+		(property "Footprint" "Capacitor_SMD:C_0805_2012Metric"
 			(at 115.2652 161.29 0)
 			(effects
@@
 			)
 		)
-		(property "LCSC" "C49326648"
+		(property "LCSC" "C13967"
 			(at 114.3 157.48 0)
 			(effects
@@
 			)
 		)
-		(property "LCSC" "C48579643"
+		(property "LCSC" "C13967"
 			(at 91.44 157.48 0)
 			(effects
@@
 			)
 		)
-		(property "LCSC" "C48579643"
+		(property "LCSC" "C13967"
 			(at 102.87 157.48 0)
 			(effects
@@
 			)
 		)
-		(property "LCSC" "C2650719"
+		(property "LCSC" "C9009"
 			(at 72.39 62.23 0)
 			(effects

Commit message: Changed crystal to oscillator
Parts:
- X1: LCSC C9009 -> C22434888
Changed lines of the file:
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@@
 			)
 		)
-		(property "LCSC" "C9009"
+		(property "LCSC" "C22434888"
 			(at 72.39 62.23 0)
 			(effects
